Commit message: successfully loaded ros2  controllers

File: urdf/gazebo_plugings.xacro (robot description, xacro)
@@ -1,16 +1,26 @@
 <?xml version="1.0"?>
 <robot xmlns:xacro="http://ros.org/wiki/xacro">
-    <xacro:macro name="four_wheels_robot">
-        <gazebo reference="base_link">
-            <plugin filename="gz_ros2_control-system" name="gz_ros2_control::GazeboSimROS2ControlPlugin">
-                <parameters>$(find four_wheels_robot)/config/wheels_controllers.yaml</parameters>
+    <!-- <xacro:macro name="four_wheels_robot"> -->
+        <gazebo>
+            <plugin filename="gz-sim-diff-drive-sysytem" name="gz::sim::system::DiffDrive">
+                <!--Wheels-->
+                <right_joint>front_right_wheel_joint</right_joint>
+                <left_joint>front_left_wheel_joint</left_joint>
+                <wheel_separation>1.6</wheel_separation>
+                <wheel_diameter>0.56</wheel_diameter>
+                <max_linear_acceleration>10</max_linear_acceleration>
+                <topic>cmd_vel</cmd_vel>
+                <tf_topic>/tf</tf_topic>
+                <odom_topic>odom</odom_topic>
+                <frame_id>odom</frame_id>
+                <child_frame_id>base_footprint</child_frame_id>
+                <odom_publisher_frequency>30</odom_publisher_frequency>
+            </plugin>
+            <!-- Joint state publisher-->
+            <plugin filename="gz-sim-joint-state-publisher-system" name="gz::sim::sysytems::JointStatePublisher">
+                <topic>joint_states</topic>
+                <joint_name>front_right_wheel_joint</joint_name>
+                <joint_name>front_left_wheel_joint</joint_name>
             </plugin>
         </gazebo>
-        <!-- Optional sensors plugin -->
-        <gazebo>
-            <plugin filename="gz-sim-sensors-system" name="gz::sim::systems::Sensors">
-                <render_engine>ogre2</render_engine>
-            </plugin>
-        </gazebo>
-    </xacro:macro>
 </robot>

File: urdf/model.urdf.xacro (robot description, xacro)
@@ -5,5 +5,5 @@
     <!-- Include control definitions -->
     <xacro:include filename="$(find four_wheels_robot)/urdf/ros2_wheel_controllers.xacro"/>
-    <xacro:include filename="$(find four_wheels_robot)/urdf/gazebo_plugings.xacro"/>
+    <!-- <xacro:include filename="$(find four_wheels_robot)/urdf/gazebo_plugings.xacro"/> -->
     <xacro:macro name="wheel" params="prefix">
         <link name="${prefix}_wheel">
@@ -55,4 +55,11 @@
         </collision>
     </link>
+    <link name="base_footprint"/>
+    <joint name="base_joint" type="fixed">
+        <origin xyz="0.0 0.0 0.0" rpy="0.0 0.0 0.0"/>
+        <parent link="base_footprint"/>
+        <child link="base_link"/>
+        <axis xyz="0.0 0.0 0.0"/>
+    </joint>
     <!-- Wheels joints (adjusted z for ground contact) -->
     <xacro:macro name="wheel_joint" params="prefix x y r">
@@ -69,5 +76,5 @@
     <xacro:wheel_joint prefix="back_right"  x="-0.41" y="-0.47" r="1.57"/>
     <!-- Add ros2_control and Gazebo plugins -->
-    <xacro:four_wheels_ros2_control/>
-    <xacro:four_wheels_robot/>
+<!-- <xacro:four_wheels_control_config/>
+<xacro:four_wheels_robot/> -->
 </robot>

File: urdf/ros2_wheel_controllers.xacro (robot description, xacro)
@@ -1,26 +1,33 @@
 <?xml version="1.0"?>
 <robot xmlns:xacro="http://ros.org/wiki/xacro">
-    <xacro:macro name="four_wheels_ros2_control">
         <ros2_control name="GazeboSystem" type="system">
             <hardware>
-                <plugin>gz_ros2_control/GazeboSystem</plugin>
+                <plugin>gz_ros2_control/GazeboSimSystem</plugin>
             </hardware>
             <joint name="front_left_wheel_joint">
                 <command_interface name="velocity"/>
                 <state_interface name="velocity"/>
+                <state_interface name="position"/>
             </joint>
             <joint name="front_right_wheel_joint">
                 <command_interface name="velocity"/>
                 <state_interface name="velocity"/>
+                <state_interface name="position"/>
             </joint>
             <joint name="back_left_wheel_joint">
                 <command_interface name="velocity"/>
                 <state_interface name="velocity"/>
+                <state_interface name="position"/>
             </joint>
             <joint name="back_right_wheel_joint">
                 <command_interface name="velocity"/>
                 <state_interface name="velocity"/>
+                <state_interface name="position"/>
             </joint>
         </ros2_control>
-    </xacro:macro>
+        <gazebo>
+        <plugin filename="gz_ros2_control-system" name="gz_ros2_control::GazeboSimROS2ControlPlugin">
+            <parameters>$(find four_wheels_robot)/config/wheels_controllers.yaml</parameters>
+        </plugin>
+    </gazebo>
 </robot>

Commit message: solved the problem of robot not moving: Issue - teleop was publishing Twist msgs while the controller was expecting Stamped. I converted both to Stamp thus solving the problem

File: urdf/gazebo_plugings.xacro (robot description, xacro)
@@ -3,24 +3,23 @@
     <!-- <xacro:macro name="four_wheels_robot"> -->
         <gazebo>
-            <plugin filename="gz-sim-diff-drive-sysytem" name="gz::sim::system::DiffDrive">
-                <!--Wheels-->
-                <right_joint>front_right_wheel_joint</right_joint>
-                <left_joint>front_left_wheel_joint</left_joint>
-                <wheel_separation>1.6</wheel_separation>
-                <wheel_diameter>0.56</wheel_diameter>
-                <max_linear_acceleration>10</max_linear_acceleration>
-                <topic>cmd_vel</cmd_vel>
-                <tf_topic>/tf</tf_topic>
-                <odom_topic>odom</odom_topic>
-                <frame_id>odom</frame_id>
-                <child_frame_id>base_footprint</child_frame_id>
-                <odom_publisher_frequency>30</odom_publisher_frequency>
-            </plugin>
-            <!-- Joint state publisher-->
-            <plugin filename="gz-sim-joint-state-publisher-system" name="gz::sim::sysytems::JointStatePublisher">
-                <topic>joint_states</topic>
-                <joint_name>front_right_wheel_joint</joint_name>
-                <joint_name>front_left_wheel_joint</joint_name>
+            <plugin filename="libgz_ros2_control-system.so" name="gz_ros2_control::GazeboSimROS2ControlPlugin">
+                <parameters>$(find four_wheels_robot)/config/wheels_controllers.yaml</parameters>
             </plugin>
         </gazebo>
+<!-- <gazebo>
+  <plugin
+      filename="libgz_ros2_control-system.so"
+      name="gz_ros2_control::GazeboSimROS2ControlPlugin">
+    <parameters>
+      $(find four_wheels_robot)/config/wheels_controllers.yaml
+    </parameters>
+  </plugin>
+</gazebo> -->
+        <!-- Optional sensors plugin <
+        <gazebo>
+            <plugin filename="gz-sim-sensors-system" name="gz::sim::systems::Sensors">
+                <render_engine>ogre2</render_engine>
+            </plugin>
+        </gazebo> -->
+    <!-- </xacro:macro> -->
 </robot>

File: urdf/model.urdf.xacro (robot description, xacro)
@@ -5,13 +5,12 @@
     <!-- Include control definitions -->
     <xacro:include filename="$(find four_wheels_robot)/urdf/ros2_wheel_controllers.xacro"/>
-    <!-- <xacro:include filename="$(find four_wheels_robot)/urdf/gazebo_plugings.xacro"/> -->
     <xacro:macro name="wheel" params="prefix">
         <link name="${prefix}_wheel">
             <inertial>
-                <origin xyz="0.0 0.0 0.0" rpy="0.0 0.0 0.0"/>
                 <mass value="0.2"/>
                 <inertia ixx="0.004087" ixy="0.0" ixz="0.0" iyy="0.004087" iyz="0.0" izz="0.007840"/>
             </inertial>
             <visual>
+                <origin xyz="0.0 0.0 0.0" rpy="1.57 0.0 0.0"/>
                 <geometry>
                     <cylinder radius="${wheel_radius}" length="${wheel_length}"/>
@@ -22,4 +21,5 @@
             </visual>
             <collision>
+             <origin xyz="0.0 0.0 0.0" rpy="1.57 0.0 0.0"/>
                 <geometry>
                     <cylinder radius="${wheel_radius}" length="${wheel_length}"/>
@@ -68,13 +68,11 @@
             <parent link="base_link"/>
             <child link="${prefix}_wheel"/>
-            <axis xyz="0 0 1"/>
+            <axis xyz="0 1 0"/>
+            <dynamics damping="0.1" friction="0.0"/>
         </joint>
     </xacro:macro>
-    <xacro:wheel_joint prefix="front_left"  x="0.41" y="0.47" r="-1.57"/>
-    <xacro:wheel_joint prefix="front_right" x="0.41" y="-0.47" r="1.57"/>
-    <xacro:wheel_joint prefix="back_left"   x="-0.41" y="0.47" r="-1.57"/>
-    <xacro:wheel_joint prefix="back_right"  x="-0.41" y="-0.47" r="1.57"/>
-    <!-- Add ros2_control and Gazebo plugins -->
-<!-- <xacro:four_wheels_control_config/>
-<xacro:four_wheels_robot/> -->
+    <xacro:wheel_joint prefix="front_left"  x="0.41" y="0.46" r="0"/>
+    <xacro:wheel_joint prefix="front_right" x="0.41" y="-0.46" r="0"/>
+    <xacro:wheel_joint prefix="back_left"   x="-0.41" y="0.46" r="0"/>
+    <xacro:wheel_joint prefix="back_right"  x="-0.41" y="-0.46" r="0"/>
 </robot>
