Commit message: successfully added lidar sensor

File: urdf/model.urdf.xacro (robot description, xacro)
@@ -5,4 +5,5 @@
     <!-- Include control definitions -->
     <xacro:include filename="$(find four_wheels_robot)/urdf/ros2_wheel_controllers.xacro"/>
+    <xacro:include filename="$(find four_wheels_robot)/urdf/sensors.xacro"/>
     <xacro:macro name="wheel" params="prefix">
         <link name="${prefix}_wheel">
@@ -76,3 +77,21 @@
     <xacro:wheel_joint prefix="back_left"   x="-0.41" y="0.46" r="0"/>
     <xacro:wheel_joint prefix="back_right"  x="-0.41" y="-0.46" r="0"/>
+    <!--Adding a lidar-->
+    <link name="lidar_link">
+        <visual>
+            <geometry>
+                <cylinder radius="0.1" length="0.08"/>
+            </geometry>
+                <material name="">
+                    <color rgba="0.78 0.55 0.34 1.0"/>
+                </material>
+        </visual>
+    </link>
+    <joint name="liadar_joint" type="fixed">
+        <origin xyz="0.0 0.0 0.2" rpy="0.0 0.0 0.0"/>
+        <parent link="base_link"/>
+        <child link="lidar_link"/>
+        <axis xyz="0.0 0.0 0.0"/>
+        <limit lower="0.0" upper="0.0" effort="0.0" velocity="0.0"/>
+    </joint>
 </robot>

Commit message: added nav2

File: urdf/model.urdf.xacro (robot description, xacro)
@@ -95,3 +95,22 @@
         <limit lower="0.0" upper="0.0" effort="0.0" velocity="0.0"/>
     </joint>
+    <!-- Adding IMU SENSOR-->
+<!-- Adding IMU SENSOR -->
+<link name="imu_link">
+  <visual>
+    <geometry>
+      <box size="0.1 0.1 0.1"/>
+    </geometry>
+  </visual>
+  <collision>
+    <geometry>
+      <box size="0.1 0.1 0.1"/>
+    </geometry>
+  </collision>
+</link>
+<joint name="imu_joint" type="fixed">
+  <parent link="base_link"/>
+  <child link="imu_link"/>
+  <origin xyz="0.0 0.0 0.0" rpy="0.0 0.0 0.0"/>
+</joint>
 </robot>

File: urdf/sensors.xacro (robot description, xacro)
@@ -11,5 +11,5 @@
             <pose relative_to='lidar_link'>0 0 0 0 0 0</pose>
             <topic>/scan</topic>
-            <update_rate>2</update_rate>
+            <update_rate>20</update_rate>
             <lidar>
                 <scan>
@@ -36,3 +36,67 @@
         </sensor>
     </gazebo>
+        <!--===========IMU SENSOR=================-->
+<gazebo reference="imu_link">
+  <sensor name="imu_sensor" type="imu">
+    <always_on>true</always_on>
+    <update_rate>10</update_rate>
+    <visualize>true</visualize>
+    <topic>/data/imu</topic>
+    <gz_frame_id>imu_link</gz_frame_id>
+    <imu>
+      <angular_velocity>
+        <x>
+          <noise type="gaussian">
+            <mean>0.0</mean>
+            <stddev>2e-4</stddev>
+            <bias_mean>0.0000075</bias_mean>
+            <bias_stddev>0.0000008</bias_stddev>
+          </noise>
+        </x>
+        <y>
+          <noise type="gaussian">
+            <mean>0.0</mean>
+            <stddev>2e-4</stddev>
+            <bias_mean>0.0000075</bias_mean>
+            <bias_stddev>0.0000008</bias_stddev>
+          </noise>
+        </y>
+        <z>
+          <noise type="gaussian">
+            <mean>0.0</mean>
+            <stddev>2e-4</stddev>
+            <bias_mean>0.0000075</bias_mean>
+            <bias_stddev>0.0000008</bias_stddev>
+          </noise>
+        </z>
+      </angular_velocity>
+      <linear_acceleration>
+        <x>
+          <noise type="gaussian">
+            <mean>0.0</mean>
+            <stddev>1.7e-2</stddev>
+            <bias_mean>0.1</bias_mean>
+            <bias_stddev>0.001</bias_stddev>
+          </noise>
+        </x>
+        <y>
+          <noise type="gaussian">
+            <mean>0.0</mean>
+            <stddev>1.7e-2</stddev>
+            <bias_mean>0.1</bias_mean>
+            <bias_stddev>0.001</bias_stddev>
+          </noise>
+        </y>
+        <z>
+          <noise type="gaussian">
+            <mean>0.0</mean>
+            <stddev>1.7e-2</stddev>
+            <bias_mean>0.1</bias_mean>
+            <bias_stddev>0.001</bias_stddev>
+          </noise>
+        </z>
+      </linear_acceleration>
+    </imu>
+  </sensor>
+</gazebo>
 </robot>

Commit message: fixed the bug, IMU now publishes it's data

File: urdf/model.urdf.xacro (robot description, xacro)
@@ -1,4 +1,4 @@
-<?xml version="1.0"?>
-<robot xmlns:xacro="http://ros.org" name="four_wheels_robot">
+<?xml version="1.1"?>
+<robot xmlns:xacro="http://ros.org/wiki/xacro" name="four_wheels_robot">
     <xacro:property name="wheel_radius" value="0.28"/>
     <xacro:property name="wheel_length" value="0.1"/>
@@ -96,5 +96,4 @@
     </joint>
     <!-- Adding IMU SENSOR-->
-<!-- Adding IMU SENSOR -->
 <link name="imu_link">
   <visual>
@@ -108,9 +107,14 @@
     </geometry>
   </collision>
+  <inertial>
+    <origin xyz="0.0 0.0 0.0" rpy="0.0 0.0 0.0"/>
+    <mass value="0.1"/>
+    <inertia ixx="0.002" ixy="0.0" ixz="0.002" iyy="0.002" iyz="0.0" izz="0.002"/>
+  </inertial>
 </link>
 <joint name="imu_joint" type="fixed">
   <parent link="base_link"/>
   <child link="imu_link"/>
-  <origin xyz="0.0 0.0 0.0" rpy="0.0 0.0 0.0"/>
+  <origin xyz="0.0 0.0 0.005" rpy="0.0 0.0 0.0"/>
 </joint>
 </robot>

File: urdf/ros2_wheel_controllers.xacro (robot description, xacro)
@@ -25,9 +25,22 @@
                 <state_interface name="position"/>
             </joint>
+            <!--IMU SENSOR-->
+             <sensor name="imu_sensor">
+                <state_interface name="orientation.x"/>
+                <state_interface name="orientation.y"/>
+                <state_interface name="orientation.z"/>
+                <state_interface name="orientation.w"/>
+                <state_interface name="angular_velocity.x"/>
+                <state_interface name="angular_velocity.y"/>
+                <state_interface name="angular_velocity.z"/>
+                <state_interface name="linear_acceleration.x"/>
+                <state_interface name="linear_acceleration.y"/>
+                <state_interface name="linear_acceleration.z"/>
+            </sensor>
         </ros2_control>
-        <gazebo>
-        <plugin filename="gz_ros2_control-system" name="gz_ros2_control::GazeboSimROS2ControlPlugin">
-            <parameters>$(find four_wheels_robot)/config/wheels_controllers.yaml</parameters>
-        </plugin>
-    </gazebo>
+    <gazebo>
+      <plugin filename="gz_ros2_control-system" name="gz_ros2_control::GazeboSimROS2ControlPlugin">
+          <parameters>$(find four_wheels_robot)/config/wheels_controllers.yaml</parameters>
+      </plugin>
+      </gazebo>
 </robot>

File: urdf/sensors.xacro (robot description, xacro)
@@ -1,10 +1,10 @@
 <?xml version="1.0"?>
 <robot xmlns:xacro="http://ros.org/wiki/xacro">
-    <!--lidar sensor-->
     <gazebo>
         <plugin filename="gz-sim-sensors-system" name="gz::sim::systems::Sensors">
             <render_engine>ogre2</render_engine>
         </plugin>
-    </gazebo>
+  </gazebo>
+        <!--lidar sensor-->
     <gazebo reference="lidar_link">
         <sensor name="gpu_lidar" type="gpu_lidar">
@@ -38,65 +38,28 @@
         <!--===========IMU SENSOR=================-->
 <gazebo reference="imu_link">
-  <sensor name="imu_sensor" type="imu">
-    <always_on>true</always_on>
-    <update_rate>10</update_rate>
-    <visualize>true</visualize>
-    <topic>/data/imu</topic>
-    <gz_frame_id>imu_link</gz_frame_id>
-    <imu>
+   <sensor name="imu_sensor" type="imu">
+      <always_on>true</always_on>
+      <update_rate>100</update_rate>
+      <noise type="gaussian">
+        <mean>0.0</mean>
+        <stddev>0.02</stddev> <!-- accelerometer noise (m/s^2) -->
+      </noise>
       <angular_velocity>
-        <x>
-          <noise type="gaussian">
-            <mean>0.0</mean>
-            <stddev>2e-4</stddev>
-            <bias_mean>0.0000075</bias_mean>
-            <bias_stddev>0.0000008</bias_stddev>
-          </noise>
-        </x>
-        <y>
-          <noise type="gaussian">
-            <mean>0.0</mean>
-            <stddev>2e-4</stddev>
-            <bias_mean>0.0000075</bias_mean>
-            <bias_stddev>0.0000008</bias_stddev>
-          </noise>
-        </y>
-        <z>
-          <noise type="gaussian">
-            <mean>0.0</mean>
-            <stddev>2e-4</stddev>
-            <bias_mean>0.0000075</bias_mean>
-            <bias_stddev>0.0000008</bias_stddev>
-          </noise>
-        </z>
+        <noise type="gaussian">
+          <mean>0.0</mean>
+          <stddev>0.001</stddev> <!-- gyro noise (rad/s) -->
+        </noise>
       </angular_velocity>
       <linear_acceleration>
-        <x>
-          <noise type="gaussian">
-            <mean>0.0</mean>
-            <stddev>1.7e-2</stddev>
-            <bias_mean>0.1</bias_mean>
-            <bias_stddev>0.001</bias_stddev>
-          </noise>
-        </x>
-        <y>
-          <noise type="gaussian">
-            <mean>0.0</mean>
-            <stddev>1.7e-2</stddev>
-            <bias_mean>0.1</bias_mean>
-            <bias_stddev>0.001</bias_stddev>
-          </noise>
-        </y>
-        <z>
-          <noise type="gaussian">
-            <mean>0.0</mean>
-            <stddev>1.7e-2</stddev>
-            <bias_mean>0.1</bias_mean>
-            <bias_stddev>0.001</bias_stddev>
-          </noise>
-        </z>
+        <noise type="gaussian">
+          <mean>0.0</mean>
+          <stddev>0.02</stddev> <!-- accel noise (m/s^2) -->
+        </noise>
       </linear_acceleration>
-    </imu>
-  </sensor>
+      <plugin filename="gz-sim-imu-system"
+              name="gz::sim::systems::Imu">
+        <topic>/imu</topic>
+      </plugin>
+    </sensor>
 </gazebo>
 </robot>
