Commit message: slam_toolbox is now working. fixed the rror discarding message by setting ros bridge and static transform between base_footprint and four_wheels_robot/base_footprint/lidar_link. map and scan now publishes well

File: urdf/model.urdf.xacro (robot description, xacro)
@@ -56,5 +56,5 @@
         </collision>
     </link>
-    <link name="base_footprint"/>
+    <link name="base_footprint"></link>
     <joint name="base_joint" type="fixed">
         <origin xyz="0.0 0.0 0.0" rpy="0.0 0.0 0.0"/>
@@ -93,5 +93,4 @@
         <child link="lidar_link"/>
         <axis xyz="0.0 0.0 0.0"/>
-        <limit lower="0.0" upper="0.0" effort="0.0" velocity="0.0"/>
     </joint>
     <!-- Adding IMU SENSOR-->

File: urdf/sensors.xacro (robot description, xacro)
@@ -7,38 +7,39 @@
   </gazebo>
         <!--lidar sensor-->
-    <gazebo reference="lidar_link">
-        <sensor name="gpu_lidar" type="gpu_lidar">
-            <pose relative_to='lidar_link'>0 0 0 0 0 0</pose>
-            <topic>/scan</topic>
-            <update_rate>20</update_rate>
-            <lidar>
-                <scan>
-                    <horizontal>
-                        <samples>720</samples>
-                        <resolution>1</resolution>
-                        <min_angle>-3.14</min_angle>
-                        <max_angle>3.14</max_angle>
-                    </horizontal>
-                </scan>
-                <range>
-                    <min>0.01</min>
-                    <max>12.0</max>
-                    <resolution>0.005</resolution>
-                </range>
-                <noise>
-                    <type>gaussian</type>
-                    <mean>0.0</mean>
-                    <stddev>0.001</stddev>
-                </noise>
-            </lidar>
-           <always_on>1</always_on>
-           <visualize>1</visualize>
-        </sensor>
-    </gazebo>
+<gazebo reference="lidar_link">
+    <sensor name="lidar_link" type="gpu_lidar">
+        <pose relative_to='lidar_link'>0 0 0 0 0 0</pose>
+        <topic>/scan</topic>
+        <update_rate>20</update_rate>
+        <frame_id>lidar_link</frame_id>
+        <lidar>
+            <scan>
+                <horizontal>
+                    <samples>720</samples>
+                    <resolution>1</resolution>
+                    <min_angle>-3.14</min_angle>
+                    <max_angle>3.14</max_angle>
+                </horizontal>
+            </scan>
+            <range>
+                <min>0.01</min>
+                <max>12.0</max>
+                <resolution>0.005</resolution>
+            </range>
+            <noise>
+                <type>gaussian</type>
+                <mean>0.0</mean>
+                <stddev>0.001</stddev>
+            </noise>
+        </lidar>
+       <always_on>1</always_on>
+       <visualize>1</visualize>
+    </sensor>
+</gazebo>
         <!--===========IMU SENSOR=================-->
 <gazebo reference="imu_link">
    <sensor name="imu_sensor" type="imu">
       <always_on>true</always_on>
-      <update_rate>100</update_rate>
+      <update_rate>20</update_rate>
       <noise type="gaussian">
         <mean>0.0</mean>

Commit message: write new nav2 params

File: urdf/model.urdf.xacro (robot description, xacro)
@@ -61,5 +61,5 @@
         <parent link="base_footprint"/>
         <child link="base_link"/>
-        <axis xyz="0.0 0.0 0.0"/>
+        <axis xyz="0.0 0.0 0.02"/>
     </joint>
     <!-- Wheels joints (adjusted z for ground contact) -->

Commit message: added new map and changed footprint at costmap

File: urdf/model.urdf.xacro (robot description, xacro)
@@ -37,5 +37,5 @@
         <inertial>
             <origin xyz="0.0 0.0 0.0" rpy="0.0 0.0 0.0"/>
-            <mass value="10.0"/> <!-- Increased mass a bit -->
+            <mass value="10.0"/>
             <inertia ixx="1.0" ixy="0.0" ixz="0.0" iyy="1.0" iyz="0.0" izz="1.0"/>
         </inertial>
@@ -63,5 +63,4 @@
         <axis xyz="0.0 0.0 0.02"/>
     </joint>
-    <!-- Wheels joints (adjusted z for ground contact) -->
     <xacro:macro name="wheel_joint" params="prefix x y r">
         <joint name="${prefix}_wheel_joint" type="continuous">

Commit message: controlling motor

File: urdf/model.urdf.xacro (robot description, xacro)
@@ -5,5 +5,5 @@
     <!-- Include control definitions -->
     <xacro:include filename="$(find four_wheels_robot)/urdf/ros2_wheel_controllers.xacro"/>
-    <xacro:include filename="$(find four_wheels_robot)/urdf/sensors.xacro"/>
+    <!-- <xacro:include filename="$(find four_wheels_robot)/urdf/sensors.xacro"/> -->
     <xacro:macro name="wheel" params="prefix">
         <link name="${prefix}_wheel">

File: urdf/ros2_wheel_controllers.xacro (robot description, xacro)
@@ -1,9 +1,20 @@
 <?xml version="1.0"?>
 <robot xmlns:xacro="http://ros.org/wiki/xacro">
-        <ros2_control name="GazeboSystem" type="system">
+        <ros2_control name="diffbot_ros2_control" type="system">
             <hardware>
-                <plugin>gz_ros2_control/GazeboSimSystem</plugin>
+                <plugin>diffdrive_arduino/DiffDriveArduinoHardware</plugin>
+                <param name="left_wheel_name">back_left_wheel_joint</param>
+                <param name="right_wheel_name">back_right_wheel_joint</param>
+                <param name="loop_rate">30</param>
+                <param name="device">/dev/ttyACM0</param>
+                <param name="baud_rate">9600</param>
+                <param name="timeout_ms">1000</param>
+                <param name="enc_counts_per_rev">3436</param>
+                <param name="pid_p">20</param>
+                <param name="pid_d">12</param>
+                <param name="pid_i">0</param>
+                <param name="pid_o">50</param>
             </hardware>
-            <joint name="front_left_wheel_joint">
+            <!-- <joint name="front_left_wheel_joint">
                 <command_interface name="velocity"/>
                 <state_interface name="velocity"/>
@@ -14,17 +25,17 @@
                 <state_interface name="velocity"/>
                 <state_interface name="position"/>
-            </joint>
+            </joint> -->
             <joint name="back_left_wheel_joint">
                 <command_interface name="velocity"/>
+                <state_interface name="position"/>
                 <state_interface name="velocity"/>
-                <state_interface name="position"/>
             </joint>
             <joint name="back_right_wheel_joint">
                 <command_interface name="velocity"/>
+                <state_interface name="position"/>
                 <state_interface name="velocity"/>
-                <state_interface name="position"/>
             </joint>
             <!--IMU SENSOR-->
-             <sensor name="imu_sensor">
+             <!-- <sensor name="imu_sensor">
                 <state_interface name="orientation.x"/>
                 <state_interface name="orientation.y"/>
@@ -37,10 +48,10 @@
                 <state_interface name="linear_acceleration.y"/>
                 <state_interface name="linear_acceleration.z"/>
-            </sensor>
+            </sensor> -->
         </ros2_control>
-    <gazebo>
+    <!-- <gazebo>
       <plugin filename="gz_ros2_control-system" name="gz_ros2_control::GazeboSimROS2ControlPlugin">
           <parameters>$(find four_wheels_robot)/config/wheels_controllers.yaml</parameters>
       </plugin>
-      </gazebo>
+      </gazebo> -->
 </robot>

Commit message: fixed error of no map frame by changing from lidar_link to laser

File: urdf/model.urdf.xacro (robot description, xacro)
@@ -77,5 +77,5 @@
     <xacro:wheel_joint prefix="back_right"  x="-0.41" y="-0.46" r="0"/>
     <!--Adding a lidar-->
-    <link name="lidar_link">
+    <link name="laser">
         <visual>
             <geometry>
@@ -90,5 +90,5 @@
         <origin xyz="0.0 0.0 0.2" rpy="0.0 0.0 0.0"/>
         <parent link="base_link"/>
-        <child link="lidar_link"/>
+        <child link="laser"/>
         <axis xyz="0.0 0.0 0.0"/>
     </joint>

Commit message: update branch

File: urdf/model.urdf.xacro (robot description, xacro)
@@ -77,5 +77,5 @@
     <xacro:wheel_joint prefix="back_right"  x="-0.41" y="-0.46" r="0"/>
     <!--Adding a lidar-->
-    <link name="lidar_link">
+    <link name="laser_link">
         <visual>
             <geometry>
@@ -87,8 +87,8 @@
         </visual>
     </link>
-    <joint name="liadar_joint" type="fixed">
+    <joint name="laser_joint" type="fixed">
         <origin xyz="0.0 0.0 0.2" rpy="0.0 0.0 0.0"/>
         <parent link="base_link"/>
-        <child link="lidar_link"/>
+        <child link="laser_link"/>
         <axis xyz="0.0 0.0 0.0"/>
     </joint>

File: urdf/sensors.xacro (robot description, xacro)
@@ -7,11 +7,11 @@
   </gazebo>
         <!--lidar sensor-->
-<gazebo reference="lidar_link">
-    <sensor name="lidar_link" type="gpu_lidar">
-        <pose relative_to='lidar_link'>0 0 0 0 0 0</pose>
+<gazebo reference="laser_link">
+    <sensor name="laser_link" type="gpu_lidar">
+        <pose relative_to='laser_link'>0 0 0 0 0 0</pose>
         <topic>/scan</topic>
         <update_rate>20</update_rate>
-        <frame_id>lidar_link</frame_id>
-        <gz_frame_id>lidar_link</gz_frame_id>
+        <frame_id>laser_link</frame_id>
+        <gz_frame_id>laser_link</gz_frame_id>
         <lidar>
             <scan>

Commit message: succesfully deployed AI model on gazebo

File: urdf/model.urdf.xacro (robot description, xacro)
@@ -116,3 +116,24 @@
   <origin xyz="0.0 0.0 0.005" rpy="0.0 0.0 0.0"/>
 </joint>
+<!-- camera link-->
+ <link name="camera_link">
+    <visual>
+        <geometry>
+            <box size="0.02 0.08 0.05"/>
+        </geometry>
+        <material name="">
+                <color rgba="1.0 0.6 0.9 1.0"/>
+            </material>
+    </visual>
+    <inertial>
+        <origin xyz="0 0 0" rpy="0 0 0"/>
+        <mass value="0.01"/>
+        <inertia ixx="0.00001" ixy="0" ixz="0" iyy="0.00001" iyz="0" izz="0.00001"/>
+    </inertial>
+ </link>
+ <joint name="camera_joint" type="fixed">
+    <parent link="base_link"/>
+    <child link="camera_link"/>
+    <origin xyz="0.7 0.0 0.15" rpy="0 0 0"/>
+ </joint>
 </robot>

File: urdf/sensors.xacro (robot description, xacro)
@@ -65,3 +65,28 @@
     </sensor>
 </gazebo>
+<!-- ===========CAMERA Link============-->
+<gazebo reference="camera_link">
+  <sensor type="camera" name="cameral">
+    <update_rate>30.0</update_rate>
+    <always_on>true</always_on>
+    <topic>camera</topic>
+    <camera name="head">
+      <horizontal_fov>1.396234</horizontal_fov>
+      <image>
+        <width>800</width>
+        <height>600</height>
+        <format>R8G8B8</format>
+      </image>
+      <clip>
+        <near>0.02</near>
+        <far>300</far>
+      </clip>
+      <noise>
+        <type>gaussian</type>
+        <mean>0.0</mean>
+        <stddev>0.007</stddev>
+      </noise>
+    </camera>
+  </sensor>
+</gazebo>
 </robot>

Commit message: revisited nav2 and added behaviour_server which brought much flexibility

File: urdf/model.urdf.xacro (robot description, xacro)
@@ -1,8 +1,8 @@
 <?xml version="1.1"?>
 <robot xmlns:xacro="http://ros.org/wiki/xacro" name="four_wheels_robot">
-    <xacro:property name="wheel_radius" value="0.28"/>
-    <xacro:property name="wheel_length" value="0.1"/>
+    <xacro:property name="wheel_radius" value="0.090"/>
+    <xacro:property name="wheel_length" value="0.04"/>
     <!-- Include control definitions -->
-    <xacro:include filename="$(find four_wheels_robot)/urdf/ros2_wheel_controllers.xacro"/>
+    <!-- <xacro:include filename="$(find four_wheels_robot)/urdf/ros2_wheel_controllers.xacro"/> -->
     <xacro:include filename="$(find four_wheels_robot)/urdf/sensors.xacro"/>
     <xacro:macro name="wheel" params="prefix">
@@ -10,5 +10,5 @@
             <inertial>
                 <mass value="0.2"/>
-                <inertia ixx="0.004087" ixy="0.0" ixz="0.0" iyy="0.004087" iyz="0.0" izz="0.007840"/>
+                <inertia ixx="0.000432" ixy="0.0" ixz="0.0" iyy="0.00081" iyz="0.0" izz="0.000432"/>
             </inertial>
             <visual>
@@ -38,10 +38,10 @@
             <origin xyz="0.0 0.0 0.0" rpy="0.0 0.0 0.0"/>
             <mass value="10.0"/>
-            <inertia ixx="1.0" ixy="0.0" ixz="0.0" iyy="1.0" iyz="0.0" izz="1.0"/>
+            <inertia ixx="0.03157" ixy="0.0" ixz="0.0" iyy="0.21667" iyz="0.0" izz="0.24013"/>
         </inertial>
         <visual>
             <origin xyz="0.0 0.0 0.0" rpy="0.0 0.0 0.0"/>
             <geometry>
-                <box size="1.3 0.8 0.4"/>
+                <box size="0.5 0.18 0.1"/>
             </geometry>
             <material name="">
@@ -52,5 +52,5 @@
             <origin xyz="0.0 0.0 0.0" rpy="0.0 0.0 0.0"/>
             <geometry>
-                <box size="1.3 0.8 0.4"/>
+                <box size="0.5 0.18 0.1"/>
             </geometry>
         </collision>
@@ -72,13 +72,13 @@
         </joint>
     </xacro:macro>
-    <xacro:wheel_joint prefix="front_left"  x="0.41" y="0.46" r="0"/>
-    <xacro:wheel_joint prefix="front_right" x="0.41" y="-0.46" r="0"/>
-    <xacro:wheel_joint prefix="back_left"   x="-0.41" y="0.46" r="0"/>
-    <xacro:wheel_joint prefix="back_right"  x="-0.41" y="-0.46" r="0"/>
+    <xacro:wheel_joint prefix="front_left"  x="0.12" y="0.12" r="0"/>
+    <xacro:wheel_joint prefix="front_right" x="0.12" y="-0.12" r="0"/>
+    <xacro:wheel_joint prefix="back_left"   x="-0.12" y="0.12" r="0"/>
+    <xacro:wheel_joint prefix="back_right"  x="-0.12" y="-0.12" r="0"/>
     <!--Adding a lidar-->
     <link name="laser_link">
         <visual>
             <geometry>
-                <cylinder radius="0.1" length="0.08"/>
+                <cylinder radius="0.05" length="0.02"/>
             </geometry>
                 <material name="">
@@ -88,5 +88,5 @@
     </link>
     <joint name="laser_joint" type="fixed">
-        <origin xyz="0.0 0.0 0.2" rpy="0.0 0.0 0.0"/>
+        <origin xyz="0.0 0.0 0.05" rpy="0.0 0.0 0.0"/>
         <parent link="base_link"/>
         <child link="laser_link"/>
@@ -97,10 +97,10 @@
   <visual>
     <geometry>
-      <box size="0.1 0.1 0.1"/>
+      <box size="0.05 0.05 0.05"/>
     </geometry>
   </visual>
   <collision>
     <geometry>
-      <box size="0.1 0.1 0.1"/>
+      <box size="0.05 0.05 0.05"/>
     </geometry>
   </collision>
@@ -120,5 +120,5 @@
     <visual>
         <geometry>
-            <box size="0.02 0.08 0.05"/>
+            <box size="0.01 0.04 0.02"/>
         </geometry>
         <material name="">
@@ -135,5 +135,5 @@
     <parent link="base_link"/>
     <child link="camera_link"/>
-    <origin xyz="0.7 0.0 0.15" rpy="0 0 0"/>
+    <origin xyz="0.25 0.0 0.03" rpy="0 0 0"/>
  </joint>
 </robot>

File: urdf/sensors.xacro (robot description, xacro)
@@ -1,16 +1,54 @@
 <?xml version="1.0"?>
 <robot xmlns:xacro="http://ros.org/wiki/xacro">
-    <gazebo>
-        <plugin filename="gz-sim-sensors-system" name="gz::sim::systems::Sensors">
-            <render_engine>ogre2</render_engine>
+ <gazebo>
+        <plugin
+          filename="gz-sim-diff-drive-system"
+          name="gz::sim::systems::DiffDrive">
+<left_joint>front_left_wheel_joint</left_joint>
+<left_joint>back_left_wheel_joint</left_joint>
+<right_joint>front_right_wheel_joint</right_joint>
+<right_joint>back_right_wheel_joint</right_joint>
+          <wheel_separation>0.26</wheel_separation>
+          <wheel_radius>0.090</wheel_radius>
+          <max_linear_acceleration>10</max_linear_acceleration>
+          <topic>/cmd_vel</topic>
+      </plugin>
+      <plugin
+        filename="gz-sim-odometry-publisher-system"
+        name="gz::sim::systems::OdometryPublisher">
+        <odom_frame>odom</odom_frame>
+        <robot_base_frame>base_footprint</robot_base_frame>
+        <odom_publish_frequency>50</odom_publish_frequency>
+        <odom_topic>/odom</odom_topic>
+        <tf_topic>/tf</tf_topic>
+        <dimensions>2</dimensions>
         </plugin>
-  </gazebo>
+        <plugin filename="gz-sim-joint-state-publisher-system" name="gz::sim::systems::JointStatePublisher">
+            <topic>joint_states</topic>
+        </plugin>
+    </gazebo>
+<gazebo reference="front_left_wheel">
+  <mu1>10.0</mu1>
+  <mu2>5.0</mu2>
+</gazebo>
+<gazebo reference="front_right_wheel">
+  <mu1>10.0</mu1>
+  <mu2>5.0</mu2>
+</gazebo>
+<gazebo reference="back_left_wheel">
+  <mu1>10.0</mu1>
+  <mu2>5.0</mu2>
+</gazebo>
+<gazebo reference="back_right_wheel">
+  <mu1>10.0</mu1>
+  <mu2>5.0</mu2>
+</gazebo>
         <!--lidar sensor-->
 <gazebo reference="laser_link">
-    <sensor name="laser_link" type="gpu_lidar">
+    <sensor name="laser_sensor" type="gpu_lidar">
         <pose relative_to='laser_link'>0 0 0 0 0 0</pose>
         <topic>/scan</topic>
         <update_rate>20</update_rate>
-        <frame_id>laser_link</frame_id>
+        <!-- <frame_id>laser_link</frame_id> -->
         <gz_frame_id>laser_link</gz_frame_id>
         <lidar>
@@ -43,4 +81,6 @@
       <always_on>true</always_on>
       <update_rate>20</update_rate>
+      <frame_id>imu_link</frame_id>
+      <gz_frame_id>imu_link</gz_frame_id>
       <noise type="gaussian">
         <mean>0.0</mean>
