Commit message: add image in gitignore

File: urdf/ros2_wheel_controllers.xacro (robot description, xacro)
@@ -1,57 +1,36 @@
 <?xml version="1.0"?>
-<robot xmlns:xacro="http://ros.org/wiki/xacro">
-        <ros2_control name="diffbot_ros2_control" type="system">
-            <hardware>
-                <plugin>diffdrive_arduino/DiffDriveArduinoHardware</plugin>
-                <param name="left_wheel_name">back_left_wheel_joint</param>
-                <param name="right_wheel_name">back_right_wheel_joint</param>
-                <param name="loop_rate">30</param>
-                <param name="device">/dev/ttyACM0</param>
-                <param name="baud_rate">9600</param>
-                <param name="timeout_ms">1000</param>
-                <param name="enc_counts_per_rev">3436</param>
-                <param name="pid_p">20</param>
-                <param name="pid_d">12</param>
-                <param name="pid_i">0</param>
-                <param name="pid_o">50</param>
-            </hardware>
-            <!-- <joint name="front_left_wheel_joint">
-                <command_interface name="velocity"/>
-                <state_interface name="velocity"/>
-                <state_interface name="position"/>
-            </joint>
-            <joint name="front_right_wheel_joint">
-                <command_interface name="velocity"/>
-                <state_interface name="velocity"/>
-                <state_interface name="position"/>
-            </joint> -->
-            <joint name="back_left_wheel_joint">
-                <command_interface name="velocity"/>
-                <state_interface name="position"/>
-                <state_interface name="velocity"/>
-            </joint>
-            <joint name="back_right_wheel_joint">
-                <command_interface name="velocity"/>
-                <state_interface name="position"/>
-                <state_interface name="velocity"/>
-            </joint>
-            <!--IMU SENSOR-->
-             <!-- <sensor name="imu_sensor">
-                <state_interface name="orientation.x"/>
-                <state_interface name="orientation.y"/>
-                <state_interface name="orientation.z"/>
-                <state_interface name="orientation.w"/>
-                <state_interface name="angular_velocity.x"/>
-                <state_interface name="angular_velocity.y"/>
-                <state_interface name="angular_velocity.z"/>
-                <state_interface name="linear_acceleration.x"/>
-                <state_interface name="linear_acceleration.y"/>
-                <state_interface name="linear_acceleration.z"/>
-            </sensor> -->
-        </ros2_control>
-    <!-- <gazebo>
-      <plugin filename="gz_ros2_control-system" name="gz_ros2_control::GazeboSimROS2ControlPlugin">
-          <parameters>$(find four_wheels_robot)/config/wheels_controllers.yaml</parameters>
-      </plugin>
-      </gazebo> -->
+<robot xmlns:xacro="http://www.ros.org/wiki/xacro">
+    <ros2_control name = "Four_Wheel_Hardware" type = "system">
+			<hardware>
+				<plugin>four_wheel_hardware/DiffBotSystemHardware</plugin>
+				<param name="hw_start_duration_sec">3</param>
+				<param name="hw_stop_duration_sec">3</param>
+				<param name="serial_port">/dev/ttyUSB0</param>
+				<param name="baudrate">115200</param>
+			</hardware>
+        <!-- <joint name="front_left_joint">
+            <command_interface name = "velocity">
+            </command_interface>
+            <state_interface name = "position" />
+						<state_interface name = "velocity" />
+        </joint> -->
+        <joint name="back_left_wheel_joint">
+            <command_interface name = "velocity">
+            </command_interface>
+            <state_interface name = "position" />
+						<state_interface name = "velocity" />
+        </joint>
+        <!-- <joint name="front_right_joint">
+            <command_interface name = "velocity">
+            </command_interface>
+            <state_interface name = "position" />
+						<state_interface name = "velocity" />
+        </joint> -->
+        <joint name="back_right_wheel_joint">
+            <command_interface name = "velocity">
+            </command_interface>
+            <state_interface name = "position" />
+						<state_interface name = "velocity" />
+        </joint>
+    </ros2_control>
 </robot>
