Commit message: Mark's fixes
removing two wheel,
changing lidar to laser

File: src/four_wheels_robot/urdf/model.urdf.xacro (robot description, xacro)
@@ -5,5 +5,5 @@
     <!-- Include control definitions -->
     <xacro:include filename="$(find four_wheels_robot)/urdf/ros2_wheel_controllers.xacro"/>
-    <xacro:include filename="$(find four_wheels_robot)/urdf/sensors.xacro"/>
+    <!-- <xacro:include filename="$(find four_wheels_robot)/urdf/sensors.xacro"/> -->
     <xacro:macro name="wheel" params="prefix">
         <link name="${prefix}_wheel">
@@ -29,6 +29,6 @@
         </link>
     </xacro:macro>
-    <xacro:wheel prefix="front_left" />
-    <xacro:wheel prefix="front_right"/>
+    <!-- <xacro:wheel prefix="front_left" /> -->
+    <!-- <xacro:wheel prefix="front_right"/> -->
     <xacro:wheel prefix="back_left"/>
     <xacro:wheel prefix="back_right" />
@@ -72,10 +72,10 @@
         </joint>
     </xacro:macro>
-    <xacro:wheel_joint prefix="front_left"  x="0.41" y="0.46" r="0"/>
-    <xacro:wheel_joint prefix="front_right" x="0.41" y="-0.46" r="0"/>
+    <!-- <xacro:wheel_joint prefix="front_left"  x="0.41" y="0.46" r="0"/> -->
+    <!-- <xacro:wheel_joint prefix="front_right" x="0.41" y="-0.46" r="0"/> -->
     <xacro:wheel_joint prefix="back_left"   x="-0.41" y="0.46" r="0"/>
     <xacro:wheel_joint prefix="back_right"  x="-0.41" y="-0.46" r="0"/>
     <!--Adding a lidar-->
-    <link name="lidar_link">
+    <link name="laser">
         <visual>
             <geometry>
@@ -90,5 +90,5 @@
         <origin xyz="0.0 0.0 0.2" rpy="0.0 0.0 0.0"/>
         <parent link="base_link"/>
-        <child link="lidar_link"/>
+        <child link="laser"/>
         <axis xyz="0.0 0.0 0.0"/>
     </joint>

Commit message: Kol is GOAT, NeovimBTW

File: src/four_wheels_robot/urdf/model.urdf.xacro (robot description, xacro)
@@ -1,6 +1,6 @@
 <?xml version="1.1"?>
 <robot xmlns:xacro="http://ros.org/wiki/xacro" name="four_wheels_robot">
-    <xacro:property name="wheel_radius" value="0.28"/>
-    <xacro:property name="wheel_length" value="0.1"/>
+    <xacro:property name="wheel_radius" value="0.090"/>
+    <xacro:property name="wheel_length" value="0.04"/>
     <!-- Include control definitions -->
     <xacro:include filename="$(find four_wheels_robot)/urdf/ros2_wheel_controllers.xacro"/>
@@ -10,5 +10,5 @@
             <inertial>
                 <mass value="0.2"/>
-                <inertia ixx="0.004087" ixy="0.0" ixz="0.0" iyy="0.004087" iyz="0.0" izz="0.007840"/>
+                <inertia ixx="0.000432" ixy="0.0" ixz="0.0" iyy="0.00081" iyz="0.0" izz="0.000432"/>
             </inertial>
             <visual>
@@ -38,10 +38,10 @@
             <origin xyz="0.0 0.0 0.0" rpy="0.0 0.0 0.0"/>
             <mass value="10.0"/>
-            <inertia ixx="1.0" ixy="0.0" ixz="0.0" iyy="1.0" iyz="0.0" izz="1.0"/>
+            <inertia ixx="0.03157" ixy="0.0" ixz="0.0" iyy="0.21667" iyz="0.0" izz="0.24013"/>
         </inertial>
         <visual>
             <origin xyz="0.0 0.0 0.0" rpy="0.0 0.0 0.0"/>
             <geometry>
-                <box size="1.3 0.8 0.4"/>
+                <box size="0.5 0.18 0.1"/>
             </geometry>
             <material name="">
@@ -52,5 +52,5 @@
             <origin xyz="0.0 0.0 0.0" rpy="0.0 0.0 0.0"/>
             <geometry>
-                <box size="1.3 0.8 0.4"/>
+                <box size="0.5 0.18 0.1"/>
             </geometry>
         </collision>
@@ -72,13 +72,13 @@
         </joint>
     </xacro:macro>
-    <!-- <xacro:wheel_joint prefix="front_left"  x="0.41" y="0.46" r="0"/> -->
-    <!-- <xacro:wheel_joint prefix="front_right" x="0.41" y="-0.46" r="0"/> -->
-    <xacro:wheel_joint prefix="back_left"   x="-0.41" y="0.46" r="0"/>
-    <xacro:wheel_joint prefix="back_right"  x="-0.41" y="-0.46" r="0"/>
+    <!-- <xacro:wheel_joint prefix="front_left"  x="0.12" y="0.12" r="0"/> -->
+    <!-- <xacro:wheel_joint prefix="front_right" x="0.12" y="-0.12" r="0"/> -->
+    <xacro:wheel_joint prefix="back_left"   x="-0.12" y="0.12" r="0"/>
+    <xacro:wheel_joint prefix="back_right"  x="-0.12" y="-0.12" r="0"/>
     <!--Adding a lidar-->
-    <link name="laser">
+    <link name="laser_link">
         <visual>
             <geometry>
-                <cylinder radius="0.1" length="0.08"/>
+                <cylinder radius="0.05" length="0.02"/>
             </geometry>
                 <material name="">
@@ -87,8 +87,8 @@
         </visual>
     </link>
-    <joint name="liadar_joint" type="fixed">
-        <origin xyz="0.0 0.0 0.2" rpy="0.0 0.0 0.0"/>
+    <joint name="laser_joint" type="fixed">
+        <origin xyz="0.0 0.0 0.05" rpy="0.0 0.0 0.0"/>
         <parent link="base_link"/>
-        <child link="laser"/>
+        <child link="laser_link"/>
         <axis xyz="0.0 0.0 0.0"/>
     </joint>
@@ -97,10 +97,10 @@
   <visual>
     <geometry>
-      <box size="0.1 0.1 0.1"/>
+      <box size="0.05 0.05 0.05"/>
     </geometry>
   </visual>
   <collision>
     <geometry>
-      <box size="0.1 0.1 0.1"/>
+      <box size="0.05 0.05 0.05"/>
     </geometry>
   </collision>
@@ -116,3 +116,24 @@
   <origin xyz="0.0 0.0 0.005" rpy="0.0 0.0 0.0"/>
 </joint>
+<!-- camera link-->
+ <link name="camera_link">
+    <visual>
+        <geometry>
+            <box size="0.01 0.04 0.02"/>
+        </geometry>
+        <material name="">
+                <color rgba="1.0 0.6 0.9 1.0"/>
+            </material>
+    </visual>
+    <inertial>
+        <origin xyz="0 0 0" rpy="0 0 0"/>
+        <mass value="0.01"/>
+        <inertia ixx="0.00001" ixy="0" ixz="0" iyy="0.00001" iyz="0" izz="0.00001"/>
+    </inertial>
+ </link>
+ <joint name="camera_joint" type="fixed">
+    <parent link="base_link"/>
+    <child link="camera_link"/>
+    <origin xyz="0.25 0.0 0.03" rpy="0 0 0"/>
+ </joint>
 </robot>
